Commit message: sync latest

File: data/project_ws/src/ros_gz_example_description/models/diff_drive_urdf/depr/model.urdf (robot description, URDF)
Before this commit: robot diff_drive, 7 links, 6 joints
Links:
- link caster: geometry collision sphere radius=0.05; visual sphere radius=0.05
- link chassis: geometry collision box size=0.3 0.3 0.15; visual box size=0.3 0.3 0.15
- link left_wheel: geometry collision cylinder length=0.03 radius=0.05; visual cylinder length=0.03 radius=0.05
- link right_wheel: geometry collision cylinder length=0.03 radius=0.05; visual cylinder length=0.03 radius=0.05
Joints:
- joint camera_joint: origin xyz=0.10 0 0.2 rpy=0 0 0 -> xyz=0.15 0 0.2 rpy=0 0 0
- joint caster_wheel: origin xyz=-0.10 0 0.10 rpy=0 0 0 -> xyz=-0.15 0 0.10 rpy=0 0 0
- joint left_wheel_joint: origin xyz=0.05 0.11 0.10 rpy=-1.5707 0 0 -> xyz=0.05 0.15 0.10 rpy=-1.5707 0 0
- joint lidar_joint: origin xyz=0 0 0.25 rpy=0 0 3.14 -> xyz=0 0 0.25 rpy=0 0 0
- joint right_wheel_joint: origin xyz=0.05 -0.11 0.10 rpy=-1.5707 0 0 -> xyz=0.05 -0.15 0.10 rpy=-1.5707 0 0

File: data/project_ws/src/ros_gz_example_description/models/diff_drive_urdf/depr/model_gazebo.urdf (robot description, URDF)
Before this commit: robot diff_drive, 7 links, 6 joints
Links:
- link caster: geometry collision sphere radius=0.05; visual sphere radius=0.05
- link chassis: geometry collision box size=0.3 0.3 0.15; visual box size=0.3 0.3 0.15
- link left_wheel: geometry collision cylinder length=0.03 radius=0.05; visual cylinder length=0.03 radius=0.05
- link right_wheel: geometry collision cylinder length=0.03 radius=0.05; visual cylinder length=0.03 radius=0.05
Joints:
- joint camera_joint: origin xyz=0.10 0 0.2 rpy=0 0 0 -> xyz=0.15 0 0.2 rpy=0 0 0
- joint caster_wheel: origin xyz=-0.10 0 0.10 rpy=0 0 0 -> xyz=-0.15 0 0.10 rpy=0 0 0
- joint left_wheel_joint: origin xyz=0.05 0.11 0.10 rpy=-1.5707 0 0 -> xyz=0.05 0.15 0.10 rpy=-1.5707 0 0
- joint lidar_joint: origin xyz=0 0 0.25 rpy=0 0 3.14 -> xyz=0 0 0.25 rpy=0 0 0
- joint right_wheel_joint: origin xyz=0.05 -0.11 0.10 rpy=-1.5707 0 0 -> xyz=0.05 -0.15 0.10 rpy=-1.5707 0 0
